File: esp_control.kicad_sch (KiCad schematic)
At the start: 5 parts, among them J1 USB_C_Receptacle_USB2.0_14P, U2 ESP32-S3-WROOM-1

Commit message: component layout, a little routing
Parts:
- renumbered R13 to R25, R11 to R26, R12 to R27
Changed lines of the file:
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@@
 		(dnp no)
 		(fields_autoplaced yes)
-		(property "Reference" "R13"
+		(property "Reference" "R25"
 			(at 179.07 34.2899 0)
 			(effects
@@
 			(project ""
 				(path "/eb928b2b-e639-4c9d-8baa-dc174c286d02/906dc8f5-0e81-43a6-aff8-165617fb8b5a"
-					(reference "R13")
+					(reference "R25")
 					(unit 1)
 				)
@@
 		(dnp no)
 		(fields_autoplaced yes)
-		(property "Reference" "#PWR031"
+		(property "Reference" "#PWR055"
 			(at 184.15 29.21 0)
 			(effects
@@
 			(project ""
 				(path "/eb928b2b-e639-4c9d-8baa-dc174c286d02/906dc8f5-0e81-43a6-aff8-165617fb8b5a"
-					(reference "#PWR031")
+					(reference "#PWR055")
 					(unit 1)
 				)
@@
 		(dnp no)
 		(fields_autoplaced yes)
-		(property "Reference" "#PWR029"
+		(property "Reference" "#PWR056"
 			(at 74.93 50.8 0)
 			(effects
@@
 			(project "oven_nametag"
 				(path "/eb928b2b-e639-4c9d-8baa-dc174c286d02/906dc8f5-0e81-43a6-aff8-165617fb8b5a"
-					(reference "#PWR029")
+					(reference "#PWR056")
 					(unit 1)
 				)
@@
 		(dnp no)
 		(fields_autoplaced yes)
-		(property "Reference" "R11"
+		(property "Reference" "R26"
 			(at 59.69 33.02 90)
 			(effects
@@
 			(project ""
 				(path "/eb928b2b-e639-4c9d-8baa-dc174c286d02/906dc8f5-0e81-43a6-aff8-165617fb8b5a"
-					(reference "R11")
+					(reference "R26")
 					(unit 1)
 				)
@@
 		(dnp no)
 		(fields_autoplaced yes)
-		(property "Reference" "R12"
+		(property "Reference" "R27"
 			(at 68.58 35.56 90)
 			(effects
@@
 			(project "oven_nametag"
 				(path "/eb928b2b-e639-4c9d-8baa-dc174c286d02/906dc8f5-0e81-43a6-aff8-165617fb8b5a"
-					(reference "R12")
+					(reference "R27")
 					(unit 1)
 				)
@@
 		(dnp no)
 		(fields_autoplaced yes)
-		(property "Reference" "#PWR030"
+		(property "Reference" "#PWR058"
 			(at 184.15 107.95 0)
 			(effects
@@
 			(project ""
 				(path "/eb928b2b-e639-4c9d-8baa-dc174c286d02/906dc8f5-0e81-43a6-aff8-165617fb8b5a"
-					(reference "#PWR030")
+					(reference "#PWR058")
 					(unit 1)
 				)
@@
 		(dnp no)
 		(fields_autoplaced yes)
-		(property "Reference" "#PWR028"
+		(property "Reference" "#PWR057"
 			(at 35.56 81.28 0)
 			(effects
@@
 			(project ""
 				(path "/eb928b2b-e639-4c9d-8baa-dc174c286d02/906dc8f5-0e81-43a6-aff8-165617fb8b5a"
-					(reference "#PWR028")
-					(unit 1)
-				)
+					(reference "#PWR057")
+					(unit 1)
+				)
