File: oven_nametag.kicad_sch (KiCad schematic)
At the start: 10 parts, among them Q1 Q_NMOS, SW1 SW_SPST, U1 TPS613221ADBV

Commit message: Added schematic
Parts:
- removed D1: LED, symbol Device:LED
- removed Q1: Q_NMOS, symbol Device:Q_NMOS
- removed R1: R, symbol Device:R
- BT1: footprint (none) -> Battery:BatteryHolder_Keystone_2466_1xAAA
- C1, C2: footprint (none) -> Capacitor_SMD:C_0805_2012Metric
- JP1: footprint (none) -> Jumper:SolderJumper-3_P1.3mm_Bridged2Bar123_Pad1.0x1.5mm_NumberLabels
- L1: footprint (none) -> Jumper:SolderJumper-3_P1.3mm_Bridged2Bar123_RoundedPad1.0x1.5mm
- SW1: footprint (none) -> Button_Switch_SMD:SW_SPDT_PCM12
Other:
- added sheet ESP Control (esp_control.kicad_sch)
- added sheet LEDs (leds.kicad_sch)
- note removed: "Boost converter: TPS613221A"
- note removed: "Times N LEDs"
- moved on the sheet: JP1

Commit message: component layout, a little routing
Parts:
- L1: footprint Jumper:SolderJumper-3_P1.3mm_Bridged2Bar123_RoundedPad1.0x1.5mm -> Inductor_SMD:L_0805_2012Metric
- renumbered C2 to C1, C1 to C2
Changed lines of the file:
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@@
 		(dnp no)
 		(fields_autoplaced yes)
-		(property "Reference" "#PWR01"
+		(property "Reference" "#PWR02"
 			(at 43.18 111.76 0)
 			(effects
@@
 			(project ""
 				(path "/eb928b2b-e639-4c9d-8baa-dc174c286d02"
-					(reference "#PWR01")
+					(reference "#PWR02")
 					(unit 1)
 				)
@@
 		(dnp no)
 		(fields_autoplaced yes)
-		(property "Reference" "#PWR02"
+		(property "Reference" "#PWR04"
 			(at 90.17 111.76 0)
 			(effects
@@
 			(project ""
 				(path "/eb928b2b-e639-4c9d-8baa-dc174c286d02"
-					(reference "#PWR02")
+					(reference "#PWR04")
 					(unit 1)
 				)
@@
 		(dnp no)
 		(fields_autoplaced yes)
-		(property "Reference" "#PWR05"
+		(property "Reference" "#PWR03"
 			(at 62.23 111.76 0)
 			(effects
@@
 			(project "oven_nametag"
 				(path "/eb928b2b-e639-4c9d-8baa-dc174c286d02"
-					(reference "#PWR05")
+					(reference "#PWR03")
 					(unit 1)
 				)
@@
 			)
 		)
-		(property "Footprint" "Jumper:SolderJumper-3_P1.3mm_Bridged2Bar123_RoundedPad1.0x1.5mm"
+		(property "Footprint" "Inductor_SMD:L_0805_2012Metric"
 			(at 72.39 86.36 0)
 			(effects
@@
 		(dnp no)
 		(fields_autoplaced yes)
-		(property "Reference" "#PWR08"
+		(property "Reference" "#PWR06"
 			(at 100.33 135.89 0)
 			(effects
@@
 			(project ""
 				(path "/eb928b2b-e639-4c9d-8baa-dc174c286d02"
-					(reference "#PWR08")
+					(reference "#PWR06")
 					(unit 1)
 				)
@@
 		(dnp no)
 		(fields_autoplaced yes)
-		(property "Reference" "#PWR03"
+		(property "Reference" "#PWR05"
 			(at 106.68 111.76 0)
 			(effects
@@
 			(project "oven_nametag"
 				(path "/eb928b2b-e639-4c9d-8baa-dc174c286d02"
-					(reference "#PWR03")
+					(reference "#PWR05")
 					(unit 1)
 				)
@@
 		(dnp no)
 		(fields_autoplaced yes)
-		(property "Reference" "#PWR04"
+		(property "Reference" "#PWR01"
 			(at 106.68 83.82 0)
 			(effects
@@
 			(project ""
 				(path "/eb928b2b-e639-4c9d-8baa-dc174c286d02"
-					(reference "#PWR04")
+					(reference "#PWR01")
 					(unit 1)
 				)
@@
 		(dnp no)
 		(fields_autoplaced yes)
-		(property "Reference" "C2"
+		(property "Reference" "C1"
 			(at 66.04 95.2499 0)
 			(effects
@@
 			(project ""
 				(path "/eb928b2b-e639-4c9d-8baa-dc174c286d02"
-					(reference "C2")
+					(reference "C1")
 					(unit 1)
 				)
@@
 		(dnp no)
 		(fields_autoplaced yes)
-		(property "Reference" "C1"
+		(property "Reference" "C2"
 			(at 110.49 95.2499 0)
 			(effects
@@
 			(project ""
 				(path "/eb928b2b-e639-4c9d-8baa-dc174c286d02"
-					(reference "C1")
-					(unit 1)
-				)
+					(reference "C2")
+					(unit 1)
+				)

Commit message: More routing
Parts:
- removed JP1: SolderJumper_3_Bridged12, Jumper:SolderJumper-3_P1.3mm_Bridged2Bar123_Pad1.0x1.5mm_NumberLabels, symbol Jumper:SolderJumper_3_Bridged12
- removed SW1: SW_SPST, Button_Switch_SMD:SW_SPDT_PCM12, symbol Switch:SW_SPST
- added RV1: 10k, Potentiometer_SMD:Potentiometer_Bourns_TC33X_Vertical, symbol Device:R_Potentiometer
- added SW2: SW_SPDT, Button_Switch_SMD:SW_SPDT_PCM12, symbol Switch:SW_SPDT
Connections:
- net +3V3: now also RV1.1
- net GND: now also RV1.3, SW2.3 (C)
- net at BT1.1 (+): now also SW2.1 (A)
- net at C1.1, L1.1: now also SW2.2 (B)
- new net LEDs/CTRL: RV1.2
Other:
- removed sheet ESP Control
- moved on the sheet: BT1
