File: leds.kicad_sch (KiCad schematic)
At the start: 30 parts, among them Q1 Q_NMOS, Q10 Q_NMOS, Q2 Q_NMOS, Q3 Q_NMOS, Q4 Q_NMOS, Q5 Q_NMOS, Q6 Q_NMOS, Q7 Q_NMOS, Q8 Q_NMOS, Q9 Q_NMOS

Commit message: component layout, a little routing
Parts:
- removed Q1, Q10, Q2, Q3, Q4, Q5, Q6, Q7, Q8, Q9: Q_NMOS, Package_TO_SOT_SMD:SOT-23, symbol Device:Q_NMOS
- added D11, D12, D13, D14, D15, D16, D17, D18, D19, D20, D21, D22, D23, D24: LED, LED_SMD:LED_1206_3216Metric, symbol Device:LED
- added Q1, Q10, Q11, Q12, Q13, Q14, Q15, Q16, Q17, Q18, Q19, Q2, Q20, Q21, Q22, Q23, Q24, Q3, Q4, Q5, Q6, Q7, Q8, Q9: BSS138, Package_TO_SOT_SMD:SOT-23, symbol Transistor_FET:BSS138
- added R11, R12, R13, R14, R15, R16, R17, R18, R19, R20, R21, R22, R23, R24: R, Resistor_SMD:R_0805_2012Metric, symbol Device:R
Connections:
- net +3V3: now also D1.2 (A), D10.2 (A), D2.2 (A), D3.2 (A), D4.2 (A), D5.2 (A), D6.2 (A), D7.2 (A), D8.2 (A), D9.2 (A), D11.2 (A), D12.2 (A), D13.2 (A), D14.2 (A), D15.2 (A), D16.2 (A), D17.2 (A), D18.2 (A), D19.2 (A), D20.2 (A), D21.2 (A), D22.2 (A), D23.2 (A), D24.2 (A); no longer R1.1, R10.1, R2.1, R3.1, R4.1, R5.1, R6.1, R7.1, R8.1, R9.1
- net CTRL: now also Q1.1 (G), Q10.1 (G), Q11.1 (G), Q12.1 (G), Q13.1 (G), Q14.1 (G), Q15.1 (G), Q16.1 (G), Q17.1 (G), Q18.1 (G), Q19.1 (G), Q2.1 (G), Q20.1 (G), Q21.1 (G), Q22.1 (G), Q23.1 (G), Q24.1 (G), Q3.1 (G), Q4.1 (G), Q5.1 (G), Q6.1 (G), Q7.1 (G), Q8.1 (G), Q9.1 (G)
- net GND: now also Q1.2 (S), Q10.2 (S), Q11.2 (S), Q12.2 (S), Q13.2 (S), Q14.2 (S), Q15.2 (S), Q16.2 (S), Q17.2 (S), Q18.2 (S), Q19.2 (S), Q2.2 (S), Q20.2 (S), Q21.2 (S), Q22.2 (S), Q23.2 (S), Q24.2 (S), Q3.2 (S), Q4.2 (S), Q5.2 (S), Q6.2 (S), Q7.2 (S), Q8.2 (S), Q9.2 (S)
- net at D10.1 (K): now also R10.1
- net at D9.1 (K): now also R9.1
- net at R1.2: now also Q1.3 (D); no longer D1.2 (A)
- net at R3.2: now also Q3.3 (D); no longer D3.2 (A)
- net at D6.1 (K): now also R6.1
- net at D2.1 (K): now also R2.1
- net at R2.2: now also Q2.3 (D); no longer D2.2 (A)
- net at R6.2: now also Q6.3 (D); no longer D6.2 (A)
- net at R9.2: now also Q9.3 (D); no longer D9.2 (A)
- net at D5.1 (K): now also R5.1
- net at R5.2: now also Q5.3 (D); no longer D5.2 (A)
- net at D7.1 (K): now also R7.1
- net at R7.2: now also Q7.3 (D); no longer D7.2 (A)
- net at D3.1 (K): now also R3.1
- net at D4.1 (K): now also R4.1
- net at R8.2: now also Q8.3 (D); no longer D8.2 (A)
- net at D1.1 (K): now also R1.1
- net at R4.2: now also Q4.3 (D); no longer D4.2 (A)
- net at R10.2: now also Q10.3 (D); no longer D10.2 (A)
- net at D8.1 (K): now also R8.1
- new net: Q21.3 (D), R21.2
- new net: D21.1 (K), R21.1
- new net: D14.1 (K), R14.1
- new net: Q14.3 (D), R14.2
- new net: Q17.3 (D), R17.2
- new net: D15.1 (K), R15.1
- new net: Q15.3 (D), R15.2
- new net: Q24.3 (D), R24.2
- new net: D20.1 (K), R20.1
- new net: D13.1 (K), R13.1
- new net: Q23.3 (D), R23.2
- new net: D17.1 (K), R17.1
- new net: D12.1 (K), R12.1
- new net: Q13.3 (D), R13.2
- new net: Q12.3 (D), R12.2
- new net: D22.1 (K), R22.1
- new net: D18.1 (K), R18.1
- new net: Q18.3 (D), R18.2
- new net: D11.1 (K), R11.1
- new net: Q11.3 (D), R11.2
- new net: D24.1 (K), R24.1
- new net: D23.1 (K), R23.1
- new net: Q16.3 (D), R16.2
- new net: Q22.3 (D), R22.2
- new net: D16.1 (K), R16.1
- new net: D19.1 (K), R19.1
- new net: Q19.3 (D), R19.2
- new net: Q20.3 (D), R20.2
Other:
- moved on the sheet: D1, D10, D2, D3, D4, D5, D6, D7, D8, D9, R1, R10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

Commit message: More routing
Connections:
- net at R9.2: no longer Q9.3 (D)
Other:
- note removed: "LEDs"
- moved on the sheet: D1, D10, D11, D12, D13, D14, D15, D16, D17, D18, D19, D2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

Commit message: Sent to pcbway
Connections:
- net at R9.2: now also Q9.3 (D)
Changed lines of the file:
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@@
+	(wire
+		(pts
+			(xy 273.05 40.64) (xy 273.05 43.18)
+		)
+		(stroke
+			(width 0)
+			(type default)
+		)
+	)
 	(wire
 		(pts
