File: oven_nametag.kicad_pcb (KiCad board)
At the start: 2 copper layers, 100 x 75 mm, 42 parts, among them J1 USB_C_Receptacle_USB2.0_14P, Q1 Q_NMOS, Q10 Q_NMOS, Q2 Q_NMOS, Q3 Q_NMOS, Q4 Q_NMOS, Q5 Q_NMOS, Q6 Q_NMOS, Q7 Q_NMOS, Q8 Q_NMOS, Q9 Q_NMOS, SW1 SW_SPST, U1 TPS613221ADBV, U2 ESP32-S3-WROOM-1

Commit message: PCB with silk option 1
Parts:
- moved BT1 154.8 mm to (31.3, 154.2)
Routing:
- added copper zone on B.Cu, net GND
- added copper zone on F.Cu, net GND
Other:
- outline, holes or cut-outs redrawn
- board text added: "My name is:"

Commit message: component layout, a little routing
Parts:
- added D11: LED, LED_SMD:LED_1206_3216Metric, F.Cu at (239.6, 68.0)
- added D12: LED, LED_SMD:LED_1206_3216Metric, F.Cu at (248.0, 68.0)
- added D13: LED, LED_SMD:LED_1206_3216Metric, F.Cu at (155.8, 105.0)
- added D14: LED, LED_SMD:LED_1206_3216Metric, F.Cu at (172.6, 105.0)
- added D15: LED, LED_SMD:LED_1206_3216Metric, F.Cu at (189.8, 105.0)
- added D16: LED, LED_SMD:LED_1206_3216Metric, F.Cu at (206.0, 105.0)
- added D17: LED, LED_SMD:LED_1206_3216Metric, F.Cu at (222.8, 105.0)
- added D18: LED, LED_SMD:LED_1206_3216Metric, F.Cu at (231.2, 105.0)
- added D19: LED, LED_SMD:LED_1206_3216Metric, F.Cu at (239.6, 105.0)
- added D20: LED, LED_SMD:LED_1206_3216Metric, F.Cu at (248.0, 105.0)
- added D21: LED, LED_SMD:LED_1206_3216Metric, F.Cu at (164.2, 105.0)
- added D22: LED, LED_SMD:LED_1206_3216Metric, F.Cu at (180.8, 105.0)
- added D23: LED, LED_SMD:LED_1206_3216Metric, F.Cu at (197.6, 105.0)
- added D24: LED, LED_SMD:LED_1206_3216Metric, F.Cu at (214.4, 105.0)
- added Q11: BSS138, Package_TO_SOT_SMD:SOT-23, F.Cu at (240.6, 60.0)
- added Q12: BSS138, Package_TO_SOT_SMD:SOT-23, F.Cu at (247.0, 60.0)
- added Q13: BSS138, Package_TO_SOT_SMD:SOT-23, F.Cu at (157.0, 55.0)
- added Q14: BSS138, Package_TO_SOT_SMD:SOT-23, F.Cu at (163.4, 55.0)
- added Q15: BSS138, Package_TO_SOT_SMD:SOT-23, F.Cu at (169.8, 55.0)
- added Q16: BSS138, Package_TO_SOT_SMD:SOT-23, F.Cu at (176.2, 55.0)
- added Q17: BSS138, Package_TO_SOT_SMD:SOT-23, F.Cu at (182.6, 55.0)
- added Q18: BSS138, Package_TO_SOT_SMD:SOT-23, F.Cu at (189.0, 55.0)
- added Q19: BSS138, Package_TO_SOT_SMD:SOT-23, F.Cu at (215.0, 55.0)
- added Q20: BSS138, Package_TO_SOT_SMD:SOT-23, F.Cu at (221.4, 55.0)
- added Q21: BSS138, Package_TO_SOT_SMD:SOT-23, F.Cu at (227.8, 55.0)
- added Q22: BSS138, Package_TO_SOT_SMD:SOT-23, F.Cu at (234.2, 55.0)
- added Q23: BSS138, Package_TO_SOT_SMD:SOT-23, F.Cu at (240.6, 55.0)
- added Q24: BSS138, Package_TO_SOT_SMD:SOT-23, F.Cu at (247.0, 55.0)
- added R11: R, Resistor_SMD:R_0805_2012Metric, F.Cu at (240.6, 63.0)
- added R12: R, Resistor_SMD:R_0805_2012Metric, F.Cu at (247.0, 63.0)
- added R13: R, Resistor_SMD:R_0805_2012Metric, F.Cu at (157.0, 52.0)
- added R14: R, Resistor_SMD:R_0805_2012Metric, F.Cu at (163.4, 52.0)
- added R15: R, Resistor_SMD:R_0805_2012Metric, F.Cu at (169.8, 52.0)
- added R16: R, Resistor_SMD:R_0805_2012Metric, F.Cu at (176.2, 52.0)
- added R17: R, Resistor_SMD:R_0805_2012Metric, F.Cu at (182.6, 52.0)
- added R18: R, Resistor_SMD:R_0805_2012Metric, F.Cu at (189.0, 52.0)
- added R19: R, Resistor_SMD:R_0805_2012Metric, F.Cu at (215.0, 52.0)
- added R20: R, Resistor_SMD:R_0805_2012Metric, F.Cu at (221.4, 52.0)
- added R21: R, Resistor_SMD:R_0805_2012Metric, F.Cu at (227.8, 52.0)
- added R22: R, Resistor_SMD:R_0805_2012Metric, F.Cu at (234.2, 52.0)
- added R23: R, Resistor_SMD:R_0805_2012Metric, F.Cu at (240.6, 52.0)
- added R24: R, Resistor_SMD:R_0805_2012Metric, F.Cu at (247.0, 52.0)
- BT1: moved to B.Cu
- L1: footprint Jumper:SolderJumper-3_P1.3mm_Bridged2Bar123_RoundedPad1.0x1.5mm -> Inductor_SMD:L_0805_2012Metric
- Q1, Q10, Q2, Q3, Q4, Q5, Q6, Q7, Q8, Q9: value Q_NMOS -> BSS138
- moved BT1 196.7 mm to (224.3, 116.1), turned to 180 degrees
- moved SW1 169.6 mm to (202.0, 122.6)
- moved C1 154.5 mm to (206.0, 59.3), turned to 90 degrees
- moved C2 146.5 mm to (198.0, 59.3), turned to 90 degrees
- moved L1 139.8 mm to (202.0, 63.1), turned to 180 degrees
- moved Q10 138.9 mm to (234.2, 60.0)
- moved U1 134.4 mm to (202.0, 59.3), turned to 90 degrees
- moved Q9 131.8 mm to (227.8, 60.0)
- moved Q8 124.7 mm to (221.4, 60.0)
- moved D10 122.7 mm to (231.2, 68.0)
- moved Q7 117.8 mm to (215.0, 60.0)
- moved R10 116.3 mm to (234.2, 63.0)
- moved D9 114.1 mm to (222.8, 68.0)
- moved R9 109.6 mm to (227.8, 63.0)
- moved D8 105.6 mm to (214.4, 68.0)
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- renumbered C2 to C1, C1 to C2, R13 to R25, R11 to R26, R12 to R27
Connections:
- D1 pad 2: Net-(D1-A) -> +3V3
- D10 pad 2: Net-(D10-A) -> +3V3
- D2 pad 2: Net-(D2-A) -> +3V3
- D3 pad 2: Net-(D3-A) -> +3V3
- D4 pad 2: Net-(D4-A) -> +3V3
- D5 pad 2: Net-(D5-A) -> +3V3
- D6 pad 2: Net-(D6-A) -> +3V3
- D7 pad 2: Net-(D7-A) -> +3V3
- D8 pad 2: Net-(D8-A) -> +3V3
- D9 pad 2: Net-(D9-A) -> +3V3
- Q1 pad 1: (no net) -> /CTRL
- Q1 pad 2: (no net) -> GND
- Q1 pad 3: (no net) -> Net-(Q1-D)
- Q10 pad 1: (no net) -> /CTRL
- Q10 pad 2: (no net) -> GND
- Q10 pad 3: (no net) -> Net-(Q10-D)
- Q2 pad 1: (no net) -> /CTRL
- Q2 pad 2: (no net) -> GND
- Q2 pad 3: (no net) -> Net-(Q2-D)
- Q3 pad 1: (no net) -> /CTRL
- Q3 pad 2: (no net) -> GND
- Q3 pad 3: (no net) -> Net-(Q3-D)
- Q4 pad 1: (no net) -> /CTRL
- Q4 pad 2: (no net) -> GND
- Q4 pad 3: (no net) -> Net-(Q4-D)
- Q5 pad 1: (no net) -> /CTRL
- Q5 pad 2: (no net) -> GND
- Q5 pad 3: (no net) -> Net-(Q5-D)
- Q6 pad 1: (no net) -> /CTRL
- Q6 pad 2: (no net) -> GND
- Q6 pad 3: (no net) -> Net-(Q6-D)
- Q7 pad 1: (no net) -> /CTRL
- Q7 pad 2: (no net) -> GND
- Q7 pad 3: (no net) -> Net-(Q7-D)
- Q8 pad 1: (no net) -> /CTRL
- Q8 pad 2: (no net) -> GND
- Q8 pad 3: (no net) -> Net-(Q8-D)
- Q9 pad 1: (no net) -> /CTRL
- Q9 pad 2: (no net) -> GND
- Q9 pad 3: (no net) -> Net-(Q9-D)
- R1 pad 1: +3V3 -> Net-(D1-K)
- R1 pad 2: Net-(D1-A) -> Net-(Q1-D)
- R10 pad 1: +3V3 -> Net-(D10-K)
- R10 pad 2: Net-(D10-A) -> Net-(Q10-D)
- R2 pad 1: +3V3 -> Net-(D2-K)
- R2 pad 2: Net-(D2-A) -> Net-(Q2-D)
- R3 pad 1: +3V3 -> Net-(D3-K)
- R3 pad 2: Net-(D3-A) -> Net-(Q3-D)
- R4 pad 1: +3V3 -> Net-(D4-K)
- R4 pad 2: Net-(D4-A) -> Net-(Q4-D)
- R5 pad 1: +3V3 -> Net-(D5-K)
- R5 pad 2: Net-(D5-A) -> Net-(Q5-D)
- R6 pad 1: +3V3 -> Net-(D6-K)
- R6 pad 2: Net-(D6-A) -> Net-(Q6-D)
- R7 pad 1: +3V3 -> Net-(D7-K)
- R7 pad 2: Net-(D7-A) -> Net-(Q7-D)
- R8 pad 1: +3V3 -> Net-(D8-K)
- R8 pad 2: Net-(D8-A) -> Net-(Q8-D)
- R9 pad 1: +3V3 -> Net-(D9-K)
- R9 pad 2: Net-(D9-A) -> Net-(Q9-D)
Routing:
- net Net-(D7-K): track 0.00 -> 11.6 mm
- net Net-(D8-K): track 0.00 -> 9.56 mm
- net Net-(D6-K): track 0.00 -> 8.36 mm
- net Net-(D9-K): track 0.00 -> 7.56 mm
- net Net-(D5-K): track 0.00 -> 6.78 mm
- net Net-(D1-K): track 0.00 -> 6.45 mm
- net Net-(D10-K): track 0.00 -> 6.44 mm
- net Net-(D4-K): track 0.00 -> 5.95 mm
- net Net-(D2-K): track 0.00 -> 5.63 mm
- net Net-(D11-K): track 0.00 -> 5.62 mm
- net Net-(D12-K): track 0.00 -> 5.21 mm
- net Net-(D3-K): track 0.00 -> 5.20 mm
- net Net-(Q9-D): track 0.00 -> 3.01 mm
- net Net-(Q8-D): track 0.00 -> 3.01 mm
- net Net-(Q7-D): track 0.00 -> 3.01 mm
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
Commit message: More routing
Parts:
- removed J1: USB_C_Receptacle_USB2.0_14P, Connector_USB:USB_C_Receptacle_GCT_USB4105-xx-A_16P_TopMnt_Horizontal
- removed JP1: SolderJumper_3_Bridged12, Jumper:SolderJumper-3_P1.3mm_Bridged2Bar123_Pad1.0x1.5mm_NumberLabels
- removed R25: 10k, Resistor_SMD:R_0805_2012Metric
- removed R26, R27: 5.1k, Resistor_SMD:R_0805_2012Metric
- removed SW1: SW_SPST, Button_Switch_SMD:SW_SPDT_PCM12
- removed U2: ESP32-S3-WROOM-1, RF_Module:ESP32-S3-WROOM-1
- added RV1: 10k, Potentiometer_SMD:Potentiometer_Bourns_TC33X_Vertical, F.Cu at (208.1, 60.8)
- added SW2: SW_SPDT, Button_Switch_SMD:SW_SPDT_PCM12, F.Cu at (202.1, 122.8)
- moved D21 58.6 mm to (222.8, 105.0)
- moved D22 50.4 mm to (231.2, 105.0)
- moved BT1 44.6 mm to (179.7, 116.0), turned to 0 degrees
- moved D23 42.0 mm to (239.6, 105.0)
- moved D17 33.6 mm to (189.2, 105.0)
- moved D18 33.6 mm to (197.6, 105.0)
- moved D19 33.6 mm to (206.0, 105.0)
- moved D20 33.6 mm to (214.4, 105.0)
- moved D24 33.6 mm to (248.0, 105.0)
- moved D16 25.2 mm to (180.8, 105.0)
- moved D15 17.2 mm to (172.6, 105.0)
- moved C1 8.87 mm to (198.0, 63.1), turned to 0 degrees
- moved D14 8.40 mm to (164.2, 105.0)
- moved L1 7.95 mm to (194.6, 60.2), turned to 90 degrees
- moved U1 3.98 mm to (198.1, 60.1), turned to 0 degrees
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Connections:
- net /CTRL renamed /LEDs/CTRL
- Q9 pad 3: Net-(Q9-D) -> unconnected-(Q9-D-Pad3)
- R9 pad 2: Net-(Q9-D) -> unconnected-(R9-Pad2)
Routing:
- net +3V3: track 0.00 -> 291.5 mm, vias 0 -> 2
- net /LEDs/CTRL: track 0.00 -> 170.3 mm
- net Net-(SW2-B): track 0.00 -> 63.8 mm, vias 0 -> 2
- net Net-(D13-K): track 0.00 -> 61.4 mm, vias 0 -> 2
- net Net-(D19-K): track 0.00 -> 60.8 mm, vias 0 -> 2
- net Net-(D20-K): track 0.00 -> 60.5 mm, vias 0 -> 2
- net Net-(D21-K): track 0.00 -> 59.2 mm, vias 0 -> 2
- net Net-(D14-K): track 0.00 -> 58.8 mm, vias 0 -> 2
- net Net-(D15-K): track 0.00 -> 58.6 mm, vias 0 -> 2
- net Net-(D18-K): track 0.00 -> 58.4 mm, vias 0 -> 2
- net Net-(D22-K): track 0.00 -> 58.4 mm, vias 0 -> 2
- net Net-(D23-K): track 0.00 -> 57.8 mm, vias 0 -> 2
- net Net-(D16-K): track 0.00 -> 57.4 mm, vias 0 -> 2
- net Net-(D17-K): track 0.00 -> 57.1 mm, vias 0 -> 2
- net Net-(D24-K): track 0.00 -> 57.1 mm, vias 0 -> 2
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
Commit message: Sent to pcbway
Parts:
- moved SW2 0.14 mm to (202.1, 122.6)
Connections:
- Q9 pad 3: unconnected-(Q9-D-Pad3) -> Net-(Q9-D)
- R9 pad 2: unconnected-(R9-Pad2) -> Net-(Q9-D)
Routing:
- net Net-(Q9-D): track 0.00 -> 3.01 mm
- net (no net): track 3.01 -> 0.00 mm
- net Net-(D19-K): track 60.8 -> 59.1 mm
- net GND: vias 29 -> 34
