File: nametag_front/nametag_front.kicad_pcb (KiCad board)
At the start: 2 copper layers, 100 x 53 mm, 4 parts

Commit message: Push new fab files
Parts:
- H1, H2, H3, H4: footprint MountingHole:MountingHole_4.3mm_M4 -> MountingHole:MountingHole_3.2mm_M3
Other:
- board text added: "r2"
Changed lines of the file:
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@@
 		(title "Two-tier nametag - front")
 		(date "2026-10-19")
-		(rev "1")
+		(rev "2")
 		(company "MAKE Roanoke")
 	)
@@
 	)
 	(net 0 "")
-	(footprint "MountingHole:MountingHole_4.3mm_M4"
+	(footprint "MountingHole:MountingHole_3.2mm_M3"
 		(layer "F.Cu")
 		(at 157 120)
-		(descr "Mounting Hole 4.3mm, M4, no annular, generated by kicad-footprint-generator mountinghole.py")
-		(tags "mountinghole M4")
+		(descr "Mounting Hole 3.2mm, M3, no annular, generated by kicad-footprint-generator mountinghole.py")
+		(tags "mountinghole M3")
 		(property "Reference" "H3"
-			(at 0 -5.25 0)
+			(at 0 -4.15 0)
 			(layer "F.SilkS")
 			(hide yes)
@@
 		)
 		(property "Value" "MountingHole"
-			(at 0 5.25 0)
-			(layer "F.Fab")
-			(effects
-				(font
-					(size 1 1)
-					(thickness 0.15)
-				)
-			)
-		)
-		(property "Datasheet" "~"
+			(at 0 4.15 0)
+			(layer "F.Fab")
+			(effects
+				(font
+					(size 1 1)
+					(thickness 0.15)
+				)
+			)
+		)
+		(property "Datasheet" ""
 			(at 0 0 0)
 			(layer "F.Fab")
@@
 			)
 		)
-		(property "Description" "Mounting Hole without connection"
+		(property "Description" ""
 			(at 0 0 0)
 			(layer "F.Fab")
@@
 		(fp_circle
 			(center 0 0)
-			(end 4.3 0)
+			(end 3.2 0)
 			(stroke
 				(width 0.15)
@@
 		(fp_circle
 			(center 0 0)
-			(end 4.55 0)
+			(end 3.45 0)
 			(stroke
 				(width 0.05)
@@
 		(pad "" np_thru_hole circle
 			(at 0 0)
-			(size 4.3 4.3)
-			(drill 4.3)
+			(size 3.2 3.2)
+			(drill 3.2)
 			(layers "*.Cu" "*.Mask")
 		)
 		(embedded_fonts no)
 	)
-	(footprint "MountingHole:MountingHole_4.3mm_M4"
+	(footprint "MountingHole:MountingHole_3.2mm_M3"
 		(layer "F.Cu")
 		(at 157 77)
-		(descr "Mounting Hole 4.3mm, M4, no annular, generated by kicad-footprint-generator mountinghole.py")
-		(tags "mountinghole M4")
+		(descr "Mounting Hole 3.2mm, M3, no annular, generated by kicad-footprint-generator mountinghole.py")
+		(tags "mountinghole M3")
 		(property "Reference" "H1"
-			(at 0 -5.25 0)
+			(at 0 -4.15 0)
 			(layer "F.SilkS")
 			(hide yes)
@@
 		)
 		(property "Value" "MountingHole"
-			(at 0 5.25 0)
-			(layer "F.Fab")
-			(hide yes)
-			(effects
-				(font
-					(size 1 1)
-					(thickness 0.15)
-				)
-			)
-		)
-		(property "Datasheet" "~"
+			(at 0 4.15 0)
+			(layer "F.Fab")
+			(effects
+				(font
+					(size 1 1)
+					(thickness 0.15)
+				)
+			)
+		)
+		(property "Datasheet" ""
 			(at 0 0 0)
 			(layer "F.Fab")
@@
 			)
 		)
-		(property "Description" "Mounting Hole without connection"
+		(property "Description" ""
 			(at 0 0 0)
 			(layer "F.Fab")
@@
 		(fp_circle
 			(center 0 0)
-			(end 4.3 0)
+			(end 3.2 0)
 			(stroke
 				(width 0.15)
@@
 		(fp_circle
 			(center 0 0)
-			(end 4.55 0)
+			(end 3.45 0)
 			(stroke
 				(width 0.05)
@@
 		(pad "" np_thru_hole circle
 			(at 0 0)
-			(size 4.3 4.3)
-			(drill 4.3)
+			(size 3.2 3.2)
+			(drill 3.2)
 			(layers "*.Cu" "*.Mask")
 		)
 		(embedded_fonts no)
 	)
-	(footprint "MountingHole:MountingHole_4.3mm_M4"
+	(footprint "MountingHole:MountingHole_3.2mm_M3"
 		(layer "F.Cu")
 		(at 247 77)
-		(descr "Mounting Hole 4.3mm, M4, no annular, generated by kicad-footprint-generator mountinghole.py")
-		(tags "mountinghole M4")
+		(descr "Mounting Hole 3.2mm, M3, no annular, generated by kicad-footprint-generator mountinghole.py")
+		(tags "mountinghole M3")
 		(property "Reference" "H2"
-			(at 0 -5.25 0)
+			(at 0 -4.15 0)
 			(layer "F.SilkS")
 			(hide yes)
@@
 		)
 		(property "Value" "MountingHole"
-			(at 0 5.25 0)
-			(layer "F.Fab")
-			(effects
-				(font
-					(size 1 1)
-					(thickness 0.15)
-				)
-			)
-		)
-		(property "Datasheet" "~"
+			(at 0 4.15 0)
+			(layer "F.Fab")
+			(effects
+				(font
+					(size 1 1)
+					(thickness 0.15)
+				)
+			)
+		)
+		(property "Datasheet" ""
 			(at 0 0 0)
 			(layer "F.Fab")
@@
 			)
 		)
-		(property "Description" "Mounting Hole without connection"
+		(property "Description" ""
 			(at 0 0 0)
 			(layer "F.Fab")
@@
 		(fp_circle
 			(center 0 0)
-			(end 4.3 0)
+			(end 3.2 0)
 			(stroke
 				(width 0.15)
@@
 		(fp_circle
 			(center 0 0)
-			(end 4.55 0)
+			(end 3.45 0)
 			(stroke
 				(width 0.05)
@@
 		(pad "" np_thru_hole circle
 			(at 0 0)
-			(size 4.3 4.3)
-			(drill 4.3)
+			(size 3.2 3.2)
+			(drill 3.2)
 			(layers "*.Cu" "*.Mask")
 		)
 		(embedded_fonts no)
 	)
-	(footprint "MountingHole:MountingHole_4.3mm_M4"
+	(footprint "MountingHole:MountingHole_3.2mm_M3"
 		(layer "F.Cu")
 		(at 247 120)
-		(descr "Mounting Hole 4.3mm, M4, no annular, generated by kicad-footprint-generator mountinghole.py")
-		(tags "mountinghole M4")
+		(descr "Mounting Hole 3.2mm, M3, no annular, generated by kicad-footprint-generator mountinghole.py")
+		(tags "mountinghole M3")
 		(property "Reference" "H4"
-			(at 0 -5.25 0)
+			(at 0 -4.15 0)
 			(layer "F.SilkS")
 			(hide yes)
@@
 		)
 		(property "Value" "MountingHole"
-			(at 0 5.25 0)
-			(layer "F.Fab")
-			(effects
-				(font
-					(size 1 1)
-					(thickness 0.15)
-				)
-			)
-		)
-		(property "Datasheet" "~"
+			(at 0 4.15 0)
+			(layer "F.Fab")
+			(effects
+				(font
+					(size 1 1)
+					(thickness 0.15)
+				)
+			)
+		)
+		(property "Datasheet" ""
 			(at 0 0 0)
 			(layer "F.Fab")
@@
 			)
 		)
-		(property "Description" "Mounting Hole without connection"
+		(property "Description" ""
 			(at 0 0 0)
 			(layer "F.Fab")
@@
 		(fp_circle
 			(center 0 0)
-			(end 4.3 0)
+			(end 3.2 0)
 			(stroke
 				(width 0.15)
@@
 		(fp_circle
 			(center 0 0)
-			(end 4.55 0)
+			(end 3.45 0)
 			(stroke
 				(width 0.05)
@@
 		(pad "" np_thru_hole circle
 			(at 0 0)
-			(size 4.3 4.3)
-			(drill 4.3)
+			(size 3.2 3.2)
+			(drill 3.2)
 			(layers "*.Cu" "*.Mask")
 		)
@@
 		)
 	)
+	(gr_text "r2"
+		(at 243.9 124.4 0)
+		(layer "B.Cu")
+		(effects
+			(font
+				(size 1.5 1.5)
+				(thickness 0.3)
+				(bold yes)
+			)
+			(justify left bottom mirror)
+		)
+	)
